Commit message: chenge the frame_id from base_foot_point to base_link

File: eg_navigation/robots/naviton_2d.urdf.xacro (robot description, xacro)
@@ -10,6 +10,6 @@
   <!-- =============== Link & Joint =============== -->
   <!-- Base -->
-  <link name="base_foot_point"/>
-  <xacro:base_v0 parent="base_foot_point">
+  <link name="base_link"/>
+  <xacro:base_v0 parent="base_link">
 	<origin xyz="0 0 0.0"/>
   </xacro:base_v0>

File: eg_navigation/robots/naviton_3d.urdf.xacro (robot description, xacro)
@@ -10,6 +10,6 @@
   <!-- =============== Link & Joint =============== -->
   <!-- Base -->
-  <link name="base_foot_point"/>
-  <xacro:base_v0 parent="base_foot_point">
+  <link name="base_link"/>
+  <xacro:base_v0 parent="base_link">
 	<origin xyz="0 0 0.0"/>
   </xacro:base_v0>

File: eg_navigation/urdf/base/base.urdf.xacro (robot description, xacro)
@@ -6,7 +6,7 @@
 	  <insert_block name="joint_origin"/>
 	  <parent link="${parent}"/>
-	  <child link="base_link"/>
+	  <child link="body_link"/>
 	</joint>
-	<link name="base_link">
+	<link name="body_link">
 	  <visual>
 		<geometry>
