Commit message: fix urdf path

File: eg_navigation/robots/naviton_3d.urdf.xacro (robot description, xacro)
@@ -1,11 +1,11 @@
 <?xml version="1.0"?>
 <robot name="naviton" xmlns:xacro="http://ros.org/wiki/xacro">
-  <xacro:include filename="$(find kcctsim)/urdf/base/base.urdf.xacro"/>
-  <xacro:include filename="$(find kcctsim)/urdf/wheel/wheel.urdf.xacro"/>
-  <xacro:include filename="$(find kcctsim)/urdf/sensors/gps/gps.urdf.xacro"/>
-  <xacro:include filename="$(find kcctsim)/urdf/sensors/gim30/gim30.urdf.xacro"/>
-  <xacro:include filename="$(find kcctsim)/urdf/sensors/lrf/lrf.urdf.xacro"/>
+  <xacro:include filename="$(find eg_navigation)/urdf/base/base.urdf.xacro"/>
+  <xacro:include filename="$(find eg_navigation)/urdf/wheel/wheel.urdf.xacro"/>
+  <xacro:include filename="$(find eg_navigation)/urdf/sensors/gps/gps.urdf.xacro"/>
+  <xacro:include filename="$(find eg_navigation)/urdf/sensors/gim30/gim30.urdf.xacro"/>
+  <xacro:include filename="$(find eg_navigation)/urdf/sensors/lrf/lrf.urdf.xacro"/>
   <xacro:include filename="$(find velodyne_description)/urdf/HDL-32E.urdf.xacro"/>
-  <xacro:include filename="$(find kcctsim)/urdf/sensors/imu/imu.urdf.xacro" />
+  <xacro:include filename="$(find eg_navigation)/urdf/sensors/imu/imu.urdf.xacro" />
   <!-- =============== Link & Joint =============== -->
   <!-- Base -->

File: eg_navigation/urdf/base/base.urdf.xacro (robot description, xacro)
@@ -1,5 +1,5 @@
 <?xml version="1.0"?>
 <robot xmlns:xacro="http://ros.org/wiki/xacro">
-  <xacro:include filename="$(find kcctsim)/urdf/base/base.gazebo.xacro"/>
+  <xacro:include filename="$(find eg_navigation)/urdf/base/base.gazebo.xacro"/>
   <xacro:macro name="base_v0" params="parent *joint_origin">
 	<joint name="base_link_joint" type="fixed">
@@ -11,6 +11,6 @@
 	  <visual>
 		<geometry>
-		 <!--- <mesh filename="package://kcctsim/meshes/DAE/base/base_link.dae"/>-->
-		 <mesh filename="package://kcctsim/meshes/STL/base/body.stl"/>
+		 <!--- <mesh filename="package://eg_navigation/meshes/DAE/base/base_link.dae"/>-->
+		 <mesh filename="package://eg_navigation/meshes/STL/base/body.stl"/>
 		</geometry>
 		<material name="gray">
@@ -20,5 +20,5 @@
 	  <collision>
 		<geometry>
-		  <mesh filename="package://kcctsim/meshes/STL/base/body.stl"/>
+		  <mesh filename="package://eg_navigation/meshes/STL/base/body.stl"/>
 		</geometry>
 	  </collision>

File: eg_navigation/urdf/sensors/gim30/gim30.urdf.xacro (robot description, xacro)
@@ -1,5 +1,5 @@
 <?xml version="1.0"?>
 <robot xmlns:xacro="http://ros.org/wiki/xacro">
-  <xacro:include filename="$(find kcctsim)/urdf/common.xacro"/>
+  <xacro:include filename="$(find eg_navigation)/urdf/common.xacro"/>
   <xacro:macro name="gim30_v0" params="parent *joint_origin">
 	<joint name="gim30_joint" type="fixed">
@@ -11,10 +11,10 @@
       <visual>
         <geometry>
-          <mesh filename="package://kcctsim/meshes/DAE/sensors/gim30/gim30.dae"/>
+          <mesh filename="package://eg_navigation/meshes/DAE/sensors/gim30/gim30.dae"/>
         </geometry>
       </visual>
 	  <collision>
 		<geometry>
-		  <mesh filename="package://kcctsim/meshes/STL/sensors/gim30/gim30.stl"/>
+		  <mesh filename="package://eg_navigation/meshes/STL/sensors/gim30/gim30.stl"/>
 		</geometry>
 	  </collision>

File: eg_navigation/urdf/sensors/gps/gps.urdf.xacro (robot description, xacro)
@@ -1,5 +1,5 @@
 <?xml version="1.0"?>
 <robot xmlns:xacro="http://ros.org/wiki/xacro">
-  <xacro:include filename="$(find kcctsim)/urdf/common.xacro"/>
+  <xacro:include filename="$(find eg_navigation)/urdf/common.xacro"/>
   <xacro:macro name="gps_v0" params="parent *joint_origin">
 	<joint name="gps_joint" type="fixed">
@@ -11,10 +11,10 @@
 	  <visual>
 		<geometry>
-		  <mesh filename="package://kcctsim/meshes/DAE/sensors/gps/gps.dae"/>
+		  <mesh filename="package://eg_navigation/meshes/DAE/sensors/gps/gps.dae"/>
 		</geometry>
 	  </visual>
 	  <collision>
 		<geometry>
-		  <mesh filename="package://kcctsim/meshes/STL/sensors/gps/gps.stl"/>
+		  <mesh filename="package://eg_navigation/meshes/STL/sensors/gps/gps.stl"/>
 		</geometry>
 	  </collision>

File: eg_navigation/urdf/sensors/lrf/lrf.urdf.xacro (robot description, xacro)
@@ -1,6 +1,6 @@
 <?xml version="1.0"?>
 <robot xmlns:xacro="http://ros.org/wiki/xacro">
-  <xacro:include filename="$(find kcctsim)/urdf/common.xacro"/>
-  <xacro:include filename="$(find kcctsim)/urdf/sensors/lrf/lrf.gazebo.xacro"/>
+  <xacro:include filename="$(find eg_navigation)/urdf/common.xacro"/>
+  <xacro:include filename="$(find eg_navigation)/urdf/sensors/lrf/lrf.gazebo.xacro"/>
   <xacro:macro name="lrf_v0" params="prefix parent *joint_origin">
 	<joint name="${prefix}_lrf_joint" type="fixed">
@@ -12,10 +12,10 @@
 	  <visual>
 		<geometry>
-		  <mesh filename="package://kcctsim/meshes/STL/sensors/utm30lx.stl"/>
+		  <mesh filename="package://eg_navigation/meshes/STL/sensors/utm30lx.stl"/>
 		</geometry>
 	  </visual>
 	  <collision>
 		<geometry>
-		  <mesh filename="package://kcctsim/meshes/STL/sensors/utm30lx.stl"/>
+		  <mesh filename="package://eg_navigation/meshes/STL/sensors/utm30lx.stl"/>
 		</geometry>
 	  </collision>

File: eg_navigation/urdf/wheel/wheel.urdf.xacro (robot description, xacro)
@@ -1,7 +1,7 @@
 <?xml version="1.0"?>
 <robot xmlns:xacro="http://ros.org/wiki/xacro">
-  <xacro:include filename="$(find kcctsim)/urdf/common.xacro"/>
-  <xacro:include filename="$(find kcctsim)/urdf/wheel/wheel.transmission.xacro"/>
-  <xacro:include filename="$(find kcctsim)/urdf/wheel/wheel.gazebo.xacro"/>
+  <xacro:include filename="$(find eg_navigation)/urdf/common.xacro"/>
+  <xacro:include filename="$(find eg_navigation)/urdf/wheel/wheel.transmission.xacro"/>
+  <xacro:include filename="$(find eg_navigation)/urdf/wheel/wheel.gazebo.xacro"/>
   <property name="wheel_radius" value="0.1575"/>
   <property name="wheel_length" value="0.032"/>
@@ -17,6 +17,6 @@
 	  <visual>
 		<geometry>
-		  <!--<mesh filename="package://kcctsim/meshes/DAE/wheel/wheel_link.dae"/>-->
-		   <mesh filename="package://kcctsim/meshes/STL/wheel/wheel.stl"/>
+		  <!--<mesh filename="package://eg_navigation/meshes/DAE/wheel/wheel_link.dae"/>-->
+		   <mesh filename="package://eg_navigation/meshes/STL/wheel/wheel.stl"/>
 		</geometry>
 		<material name="black">

Commit message: apply noetic

File: eg_navigation/robots/naviton_3d.urdf.xacro (robot description, xacro)
@@ -80,6 +80,6 @@
 					   min_range="0.10" max_range="60.0"/>
   <!-- VHDL-32E -->
-  <HDL-32E parent="base_link" name="velodyne" topic="velodyne_points" hz="10" samples="1024" gpu="true">
+  <xacro:HDL-32E parent="base_link" name="velodyne" topic="velodyne_points" hz="10" samples="1024" gpu="true">
       <origin xyz="0 0 0.8" rpy="0 0 0" />
-  </HDL-32E>
+  </xacro:HDL-32E>
 </robot>

File: eg_navigation/urdf/base/base.urdf.xacro (robot description, xacro)
@@ -4,5 +4,5 @@
   <xacro:macro name="base_v0" params="parent *joint_origin">
 	<joint name="base_link_joint" type="fixed">
-	  <insert_block name="joint_origin"/>
+	  <xacro:insert_block name="joint_origin"/>
 	  <parent link="${parent}"/>
 	  <child link="body_link"/>
@@ -15,5 +15,5 @@
 		</geometry>
 		<material name="gray">
-    <color rgba="0.8 0.8 0.8 2.0"/>
+    <color rgba="0.8 0.8 0.8 1.0"/>
   </material>
 	  </visual>

File: eg_navigation/urdf/common.xacro (robot description, xacro)
@@ -1,5 +1,5 @@
 <?xml version="1.0"?>
 <robot xmlns:xacro="http://ros.org/wiki/xacro">
-  <property name="M_PI" value="3.14159274"/>
+  <xacro:property name="M_PI" value="3.14159274"/>
   <xacro:macro name="cylinder_inertial" params="mass radius length">
 	<mass value="${mass}"/>

File: eg_navigation/urdf/sensors/gim30/gim30.urdf.xacro (robot description, xacro)
@@ -4,5 +4,5 @@
   <xacro:macro name="gim30_v0" params="parent *joint_origin">
 	<joint name="gim30_joint" type="fixed">
-      <insert_block name="joint_origin" />
+      <xacro:insert_block name="joint_origin" />
       <parent link="${parent}"/>
       <child link="gim30_link"/>
@@ -21,5 +21,5 @@
 	  <inertial>
 		<origin xyz="-0.04 0 -0.1"/>
-		<box_inertial mass="0.85" height="0.1" width="0.05" depth="0.25"/>
+		<xacro:box_inertial mass="0.85" height="0.1" width="0.05" depth="0.25"/>
 	  </inertial>
     </link>

File: eg_navigation/urdf/sensors/gps/gps.urdf.xacro (robot description, xacro)
@@ -4,5 +4,5 @@
   <xacro:macro name="gps_v0" params="parent *joint_origin">
 	<joint name="gps_joint" type="fixed">
-	  <insert_block name="joint_origin"/>
+	  <xacro:insert_block name="joint_origin"/>
 	  <parent link="${parent}"/>
 	  <child link="gps_link"/>
@@ -20,5 +20,5 @@
 	  </collision>
 	  <inertial>
-		<cylinder_inertial mass="0.25" radius="0.065" length="0.055"/>
+		<xacro:cylinder_inertial mass="0.25" radius="0.065" length="0.055"/>
 	  </inertial>
 	</link>

File: eg_navigation/urdf/sensors/lrf/lrf.urdf.xacro (robot description, xacro)
@@ -5,5 +5,5 @@
   <xacro:macro name="lrf_v0" params="prefix parent *joint_origin">
 	<joint name="${prefix}_lrf_joint" type="fixed">
-	  <insert_block name="joint_origin"/>
+	  <xacro:insert_block name="joint_origin"/>
 	  <parent link="${parent}"/>
 	  <child link="${prefix}_lrf_link"/>
@@ -22,5 +22,5 @@
 	  <inertial>
 		<origin xyz="0 0 -0.0164"/>
-		<box_inertial mass="0.4" height="0.07" width="0.07" depth="0.08"/>
+		<xacro:box_inertial mass="0.4" height="0.07" width="0.07" depth="0.08"/>
 	  </inertial>
 	</link>

File: eg_navigation/urdf/wheel/wheel.urdf.xacro (robot description, xacro)
@@ -4,13 +4,13 @@
   <xacro:include filename="$(find eg_navigation)/urdf/wheel/wheel.transmission.xacro"/>
   <xacro:include filename="$(find eg_navigation)/urdf/wheel/wheel.gazebo.xacro"/>
-  <property name="wheel_radius" value="0.1575"/>
-  <property name="wheel_length" value="0.032"/>
-  <property name="wheel_mass" value="2.0"/>
+  <xacro:property name="wheel_radius" value="0.1575"/>
+  <xacro:property name="wheel_length" value="0.032"/>
+  <xacro:property name="wheel_mass" value="2.0"/>
   <xacro:macro name="wheel_v0" params="prefix parent *joint_origin *joint_axis">
 	<joint name="${prefix}_wheel_joint" type="continuous">
-	  <insert_block name="joint_origin"/>
+	  <xacro:insert_block name="joint_origin"/>
 	  <parent link="${parent}"/>
 	  <child link="${prefix}_wheel_link"/>
-	  <insert_block name="joint_axis"/>
+	  <xacro:insert_block name="joint_axis"/>
 	</joint>
 	<link name="${prefix}_wheel_link">
@@ -21,5 +21,5 @@
 		</geometry>
 		<material name="black">
-    		<color rgba="0.2 0.2 0.2 2.0"/>
+    		<color rgba="0.2 0.2 0.2 1.0"/>
   		</material>
 	  </visual>
@@ -32,5 +32,5 @@
 	  <inertial>
 		<origin xyz="0 -0.003 0" rpy="${-M_PI/2} 0 0"/>
-		<cylinder_inertial mass="${wheel_mass}"
+		<xacro:cylinder_inertial mass="${wheel_mass}"
 						   radius="${wheel_radius}" length="${wheel_length}"/>
 	  </inertial>
